Commit message: camera is working good

File: cycloidal_arm/urdf/camera.xacro (robot description, xacro)
@@ -1,31 +1,35 @@
 <?xml version="1.0" ?>
 <robot name="cycloidal_arm" xmlns:xacro="http://www.ros.org/wiki/xacro" >
-<!-- <link name="camera_optical"/>
+<link name="camera_optical"/>
 <joint name="camera_optical_joint" type="fixed">
   <parent link="camera"/>
   <child link="camera_optical"/>
-  <origin xyz="0 0 0" rpy="0 0 0"/>
-</joint> -->
-<gazebo reference="camera">
-    <material>Gazebo/Red</material>
-    <sensor name="camera" type="camera">
-    <pose>0 0 0 0 0 0 0</pose>
-    <visualize>true</visualize>
-    <update_rate>10</update_rate>
-    <camera>
-      <horizontal_fov>1.089</horizontal_fov>
-      <image>
-        <format>R8G8B8</format>
-        <width>640</width>
-        <height>640</height>
-      </image>
-      <clip>
-        <near>0.05</near>
-        <far>8.0</far>
-      </clip>
-    </camera>
-    <puglin name="camera_controller" filename="libgazebo_ros_camera.so">
-        <frame_name>camera</frame_name>
-    </puglin>
+  <origin xyz="0 0 0" rpy="0 -1.57 1.57"/>
+</joint>
+<gazebo reference="camera_optical">
+    <sensor type="camera" name="camera">
+        <pose> 0.2 0 0 1.57 0 1.57 </pose>
+        <visualize>true</visualize>
+        <update_rate>30.0</update_rate>
+        <camera name="head">
+          <horizontal_fov>1.089</horizontal_fov>
+          <image>
+            <width>640</width>
+            <height>640</height>
+            <format>R8G8B8</format>
+          </image>
+          <clip>
+            <near>0.05</near>
+            <far>30</far>
+          </clip>
+        </camera>
+        <plugin name="camera_controller" filename="libgazebo_ros_camera.so">
+          <alwaysOn>true</alwaysOn>
+          <update_rate>0.0</update_rate>
+          <cameraName>cycloidal_arm/camera_optical</cameraName>
+          <imageTopicName>image_raw</imageTopicName>
+          <cameraInfoTopicName>camera_info</cameraInfoTopicName>
+          <frame_name>camera_optical</frame_name>
+        </plugin>
     </sensor>
 </gazebo>

File: cycloidal_arm/urdf/cycloidal_arm.xacro (robot description, xacro)
@@ -191,4 +191,4 @@
 <xacro:include filename="$(find cycloidal_arm)/urdf/arm_gazebo.xacro" />
 <xacro:include filename="$(find cycloidal_arm)/urdf/arm_trans.xacro" />
- <!-- <xacro:include filename="$(find cycloidal_arm)/urdf/camera.xacro" />   -->
+<xacro:include filename="$(find cycloidal_arm)/urdf/camera.xacro" />
 </robot>
