Commit message: Renamed some files and add the ros2_control but some are there in it

File: cycloidal_arm/urdf/cycloidal_arm.xacro (robot description, xacro)
@@ -189,6 +189,7 @@
 </joint>
 <!-- <xacro:include filename="$(find cycloidal_arm)/urdf/cycloidal_arm.trans" /> -->
-<xacro:include filename="$(find cycloidal_arm)/urdf/arm_gazebo.xacro" />
-<xacro:include filename="$(find cycloidal_arm)/urdf/arm_trans.xacro" />
+<xacro:include filename="$(find cycloidal_arm)/urdf/gazebo_arm.xacro" />
+<xacro:include filename="$(find cycloidal_arm)/urdf/trans_arm.xacro" />
 <xacro:include filename="$(find cycloidal_arm)/urdf/camera.xacro" />
+<xacro:include filename="$(find cycloidal_arm)/urdf/ros2_control.xacro"/>
 </robot>

File: cycloidal_arm/urdf/gazebo_arm.xacro (robot description, xacro)
@@ -37,3 +37,9 @@
     <selfCollide>false</selfCollide>
 </gazebo>
+<gazebo reference="camera">
+    <material>Gazebo/Red</material>
+    <mu1>0.5</mu1>
+    <mu2>0.5</mu2>
+    <selfCollide>false</selfCollide>
+</gazebo>
 </robot>
